Commit message: Refine Tiangong3 model and actuator configuration
Co-authored-by: Cursor <cursoragent@cursor.com>

File: src/assets/robots/tiangong3/urdf/tiangong3.urdf (robot description, URDF)
Before this commit: robot tiangong3, 39 links, 38 joints
Links:
- link elbow_pitch_l_link: geometry collision cylinder length=0.12 radius=0.035; visual mesh filename=../meshes_convex/elbow_pitch_l_link.STL
- link elbow_pitch_r_link: geometry collision cylinder length=0.12 radius=0.035; visual mesh filename=../meshes_convex/elbow_pitch_r_link.STL
- link hip_roll_l_link: geometry collision sphere radius=0.05; visual mesh filename=../meshes_convex/hip_roll_l_link.STL
- link hip_roll_r_link: geometry collision sphere radius=0.05; visual mesh filename=../meshes_convex/hip_roll_r_link.STL
- link hip_yaw_l_link: geometry collision cylinder length=0.18 radius=0.04; visual mesh filename=../meshes_convex/hip_yaw_l_link.STL
- link hip_yaw_r_link: geometry collision cylinder length=0.18 radius=0.04; visual mesh filename=../meshes_convex/hip_yaw_r_link.STL
- link knee_pitch_l_link: geometry collision cylinder length=0.23 radius=0.035; visual mesh filename=../meshes_convex/knee_pitch_l_link.STL
- link knee_pitch_r_link: geometry collision cylinder length=0.23 radius=0.035; visual mesh filename=../meshes_convex/knee_pitch_r_link.STL
- link shoulder_yaw_l_link: geometry visual mesh filename=../meshes_convex/shoulder_yaw_l_link.STL
- link shoulder_yaw_r_link: geometry visual mesh filename=../meshes_convex/shoulder_yaw_r_link.STL
- link wrist_pitch_l_link: geometry visual mesh filename=../meshes_convex/wrist_pitch_l_link.STL
- link wrist_pitch_r_link: geometry visual mesh filename=../meshes_convex/wrist_pitch_r_link.STL
Joints:
- joint ankle_pitch_l_joint: origin xyz=0.0073682 0 -0.39993 rpy=0 0 0 -> xyz=0.0 0 -0.4 rpy=0 0 0
- joint ankle_pitch_r_joint: origin xyz=0.014553 0 -0.39974 rpy=0 0 0 -> xyz=0.0 0 -0.4 rpy=0 0 0
- joint elbow_yaw_l_joint: type revolute -> fixed
- joint elbow_yaw_r_joint: type revolute -> fixed
- joint knee_pitch_l_joint: origin xyz=-0.012927 0 -0.30599 rpy=0 0.018418 0 -> xyz=-0.012927 0 -0.30599 rpy=0 0.0 0
- joint knee_pitch_r_joint: origin xyz=-0.012927 0 -0.30599 rpy=0 0.036386 0 -> xyz=-0.012927 0 -0.30599 rpy=0 0.0 0
- joint wrist_pitch_l_joint: type revolute -> fixed
- joint wrist_pitch_r_joint: type revolute -> fixed
- joint wrist_roll_l_joint: type revolute -> fixed
- joint wrist_roll_r_joint: type revolute -> fixed
